File: LARP Gun/Gun_Trigger.sch (EAGLE design)
At the start: 9 parts

Commit message: Updated cad files, and working sketch for the magazine
Parts:
- AMMO: device SparkFun-Connectors:M05PTH -> SparkFun-Connectors:M06POLAR
