File: Shield Generator/Sheild Generator - Main unit.brd (EAGLE design)
At the start: 81 x 63.5 mm, 40 parts, among them IC1 ATMEGA168-PU, IC2 7805T

Commit message: Updated cad files, and working sketch for the magazine
Parts:
- moved R2 1.27 mm to (96.5, 14.0)
- moved R1 1.27 mm to (86.4, 14.0)
Routing:
- net +12V: track 124.1 -> 0.00 mm
- net GND: track 16.4 -> 53.3 mm
- net N$5: track 98.0 -> 79.9 mm
- net N$28: track 32.4 -> 19.4 mm, vias 1 -> 0
- net N$3: track 67.0 -> 54.0 mm
- net N$18: track 25.1 -> 34.2 mm
- net N$23: track 36.8 -> 28.1 mm
- net +5V: track 64.2 -> 72.5 mm
- net N$26: track 24.0 -> 31.9 mm
- net N$2: track 55.8 -> 63.5 mm, vias 2 -> 0
- net N$4: track 37.4 -> 41.9 mm, vias 1 -> 0
- net N$1: track 64.9 -> 61.0 mm, vias 1 -> 0
- net N$20: track 14.0 -> 17.5 mm, vias 0 -> 1
- net N$10: track 54.8 -> 51.4 mm, vias 1 -> 2
- net N$15: track 55.8 -> 58.3 mm, vias 0 -> 1
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- added copper zone on layer 1, net +12V
