File: Shield Generator/Sheild Generator - Main unit.sch (EAGLE design)
At the start: 40 parts, among them IC1 ATMEGA168-PU, IC2 7805T

Commit message: Updated cad files, and working sketch for the magazine
Connections:
- net +5V renamed VCC
